File: pcb/backups/pre-standby/layout.kicad_pcb (KiCad board)
At the start: 2 copper layers, 115 parts, among them J1 B2B-PH-K-S, J3 B2B-PH-K-S, J4 104031-0811, Q1 AO3400A, Q2 AO3400A, SW1 PTS841GKSMTR LFS, SW2 JS202011AQN, U1 113991114, U10 SN74CBTLV3245APWR, U11 SN74CBTLV3245APWR, U3 MAX17048G+T10, U4 BMI270, U5 TPS61023DRLR, U6 AP2112K-3.3TRG1, U7 TPS22918DBVR, U8 TPS22918DBVR, U9 TPS22918DBVR

Commit message: Add compact placement candidate and update BOM, layout, and component library
Parts:
- removed C41, C42: GRM1555C1E102JA01D, stdlib_kicad-footprints_Capacitor_SMD:C_0402_1005Metric
- removed C43, C44: CC0805KRX5R8BB106, stdlib_kicad-footprints_Capacitor_SMD:C_0805_2012Metric
- removed C45, C46: GRM155R71C104KA88D, stdlib_kicad-footprints_Capacitor_SMD:C_0402_1005Metric
- removed Q2: AO3400A, embedr_ai_pendant_recorder_components_ao3400a_assets:SOT-23
- removed R29: RC0603FR-07100KL, stdlib_kicad-footprints_Resistor_SMD:R_0603_1608Metric
- removed R30: RC0603FR-074K7L, stdlib_kicad-footprints_Resistor_SMD:R_0603_1608Metric
- removed U10, U11: SN74CBTLV3245APWR, embedr_ai_pendant_recorder_components_sn74cbtlv3245a:TSSOP-20
- removed U8, U9: TPS22918DBVR, embedr_ai_pendant_recorder_components_tps22918_assets:SOT-23-6
Connections:
- C12 pad 1: VBAT_PERIPH -> VBAT
- C7 pad 1: VBAT_PERIPH -> VBAT
- L1 pad 1: VBAT_PERIPH -> VBAT
- R1 pad 2: V3V3_AON -> V3V3
- SW2 pad 4: GND -> SW2.POLE2_THROW_A
- SW2 pad 5: RUN_ENABLE -> SW2.POLE2_COMMON
- SW2 pad 6: V3V3_AON -> SW2.POLE2_THROW_B
- U1 pad 1: HOST_HAPTIC -> HAPTIC_DRIVE
- U1 pad 10: HOST_SD_MISO -> SD_MISO
- U1 pad 11: HOST_SD_MOSI -> SD_MOSI
- U1 pad 12: V3V3_AON -> V3V3
- U1 pad 15: HOST_PDM_DATA -> PDM_DATA
- U1 pad 16: HOST_IMU_INT -> IMU_INT
- U1 pad 19: HOST_PDM_CLK -> PDM_CLK_MCU
- U1 pad 20: HOST_SD_CS -> SD_CS
- U1 pad 3: HOST_LED_ENABLE -> LED_ENABLE
- U1 pad 4: HOST_LED_DATA -> LED_DATA_MCU
- U1 pad 5: HOST_SDA -> FG_SDA
- U1 pad 6: HOST_SCL -> FG_SCL
- U1 pad 9: HOST_SD_CLK -> SD_CLK_MCU
- U5 pad 3: VBAT_PERIPH -> VBAT
- U6 pad 1: VBAT_PERIPH -> VBAT
- U6 pad 3: VBAT_PERIPH -> VBAT
