File: pcb/freerouting-api-20260921/layout.width020-low-via-completed.kicad_pcb (KiCad board)
At the start: 4 copper layers, 36 x 76 mm, 115 parts, among them J1 B2B-PH-K-S, J3 B2B-PH-K-S, J4 104031-0811, Q1 AO3400A, Q2 AO3400A, SW1 PTS841GKSMTR LFS, SW2 JS202011AQN, U1 113991114, U10 SN74CBTLV3245APWR, U11 SN74CBTLV3245APWR, U3 MAX17048G+T10, U4 BMI270, U5 TPS61023DRLR, U6 AP2112K-3.3TRG1, U7 TPS22918DBVR, U8 TPS22918DBVR, U9 TPS22918DBVR

Commit message: Update board configuration, BOM, and documentation for new XIAO ESP32S3
Routing:
- net GND: track 412.7 -> 409.9 mm
Changed lines of the file:
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@@
+	)
+	(segment
+		(start 83.6 94.6)
+		(end 84.2 93.69)
+		(width 0.2)
+		(layer "F.Cu")
+		(net "GND")
 	)
 	(segment
@@
 	)
 	(segment
-		(start 86.7 93.7)
-		(end 85.68 93.69)
-		(width 0.2)
-		(layer "F.Cu")
-		(net "GND")
-	)
-	(segment
 		(start 102.085 81.55)
 		(end 102.23 81.55)
@@
 	)
 	(segment
-		(start 84.2 95.35)
-		(end 84.8 96.1)
-		(width 0.2)
-		(layer "F.Cu")
-		(net "GND")
-	)
-	(segment
 		(start 90.2048 85.6698)
 		(end 90.085 85.55)
@@
 	)
 	(segment
+		(start 84.2 93.69)
+		(end 85.68 93.69)
+		(width 0.2)
+		(layer "F.Cu")
+		(net "GND")
+	)
+	(segment
 		(start 113.9636 75.7748)
 		(end 113.2384 76.5)
@@
 	)
 	(segment
+		(start 85.68 93.69)
+		(end 87.325 93.55)
+		(width 0.2)
+		(layer "F.Cu")
+		(net "GND")
+	)
+	(segment
 		(start 98.1375 67.275)
 		(end 98.1375 66.625)
@@
 	)
 	(segment
-		(start 86.7 96.1)
-		(end 86.7 93.7)
-		(width 0.2)
-		(layer "F.Cu")
-		(net "GND")
-	)
-	(segment
 		(start 104.835 78.8)
 		(end 103.48 78.8)
@@
 	)
 	(segment
+		(start 84.2 95.35)
+		(end 83.6 94.6)
+		(width 0.2)
+		(layer "F.Cu")
+		(net "GND")
+	)
+	(segment
 		(start 95.48 82.8)
 		(end 96.835 82.8)
@@
 	)
 	(segment
-		(start 84.8 96.1)
-		(end 86.7 96.1)
-		(width 0.2)
-		(layer "F.Cu")
-		(net "GND")
-	)
-	(segment
 		(start 110 70.175)
 		(end 108.6544 68.8294)
@@
 		(width 0.2)
 		(layer "F.Cu")
-		(net "GND")
-	)
-	(segment
-		(start 85.68 93.69)
-		(end 87.325 93.55)
-		(width 0.2)
-		(layer "F.Cu")
